Commit message: Got it working with 4 wheels

File: bb1_description/urdf/bb1.urdf (robot description, URDF)
Before this commit: robot burt, 5 links, 4 joints
Joints:
- removed joint base_to_left_back_wheel_joint
- removed joint base_to_left_front_wheel_joint
- removed joint base_to_right_back_wheel_joint
- removed joint base_to_right_front_wheel_joint
- added joint back_left_wheel_joint: type continuous, parent base_link, child left_back_wheel, origin xyz=-0.09 0.12 -0.025, axis 0 1 0
- added joint back_right_wheel_joint: type continuous, parent base_link, child right_back_wheel, origin xyz=-0.09 -0.12 -0.025, axis 0 1 0
- added joint front_left_wheel_joint: type continuous, parent base_link, child left_front_wheel, origin xyz=0.09 0.12 -0.025, axis 0 1 0
- added joint front_right_wheel_joint: type continuous, parent base_link, child right_front_wheel, origin xyz=0.09 -0.12 -0.025, axis 0 1 0

Commit message: New working configuration

File: bb1_description/urdf/bb1.urdf (robot description, URDF)
Before this commit: robot burt, 5 links, 4 joints
Links:
- removed link left_back_wheel
- removed link left_front_wheel
- removed link right_back_wheel
- removed link right_front_wheel
- added link back_left_wheel, mass 3; collision cylinder length=0.045 radius=0.085; visual cylinder length=0.045 radius=0.085
- added link back_right_wheel, mass 3; collision cylinder length=0.045 radius=0.085; visual cylinder length=0.045 radius=0.085
- added link front_left_wheel, mass 3; collision cylinder length=0.045 radius=0.085; visual cylinder length=0.045 radius=0.085
- added link front_right_wheel, mass 3; collision cylinder length=0.045 radius=0.085; visual cylinder length=0.045 radius=0.085
Joints:
- joint back_left_wheel_joint: child left_back_wheel -> back_left_wheel
- joint back_right_wheel_joint: child right_back_wheel -> back_right_wheel
- joint front_left_wheel_joint: child left_front_wheel -> front_left_wheel
- joint front_right_wheel_joint: child right_front_wheel -> front_right_wheel

Commit message: Updated URDF to reflect new robot model

File: bb1_description/urdf/bb1.urdf (robot description, URDF)
Before this commit: robot burt, 5 links, 4 joints
Links:
- link base_link: mass 15 -> 1; geometry collision box size=0.30 0.25 0.058; visual box size=0.30 0.25 0.058
Joints:
- joint back_left_wheel_joint: origin xyz=-0.09 0.12 -0.025 -> xyz=-0.09 0.135 -0.035
- joint back_right_wheel_joint: origin xyz=-0.09 -0.12 -0.025 -> xyz=-0.09 -0.135 -0.035
- joint front_left_wheel_joint: origin xyz=0.09 0.12 -0.025 -> xyz=0.09 0.135 -0.035
- joint front_right_wheel_joint: origin xyz=0.09 -0.12 -0.025 -> xyz=0.09 -0.135 -0.035
